File: hw/hw.sch (KiCad schematic (older format))
At the start: 30 parts, among them J1 Motor 1 Connector, J2 Motor 2 Connector, J3 Distance sensor 2, J4 Distance sensor 1, J5 Distance sensor 3, J6 Serial pin header, J7 Distance sensor 4, J8 Distance sensor 5, U1 TB6612FNG_Breakout, U2 L3GD20_breakout

Commit message: Added PCB v1.2
Parts:
- BT1: value Battery_Cell -> Battery
- J3: value Distance sensor 2 -> sensor 2
- J4: value Distance sensor 1 -> sensor 1
- J5: value Distance sensor 3 -> sensor 3
- J6: value Serial pin header -> TX/RX
- J7: value Distance sensor 4 -> sensor 4
- J8: value Distance sensor 5 -> sensor 5
Changed lines of the file:
@@
 P 8800 3300
 F 0 "J4" H 8693 2975 50  0000 C CNN
-F 1 "Distance sensor 1" H 8693 3066 50  0000 C CNN
+F 1 "sensor 1" H 8693 3066 50  0000 C CNN
 F 2 "Connector_PinSocket_2.54mm:PinSocket_1x03_P2.54mm_Vertical" H 8800 3300 50  0001 C CNN
 F 3 "~" H 8800 3300 50  0001 C CNN
@@
 P 750 1450
 F 0 "BT1" H 868 1546 50  0000 L CNN
-F 1 "Battery_Cell" H 868 1455 50  0000 L CNN
+F 1 "Battery" H 868 1455 50  0000 L CNN
 F 2 "Connector_PinSocket_2.54mm:PinSocket_1x02_P2.54mm_Vertical" V 750 1510 50  0001 C CNN
 F 3 "~" V 750 1510 50  0001 C CNN
@@
 P 4150 3150
 F 0 "J6" H 4256 3328 50  0000 C CNN
-F 1 "Serial pin header" H 4250 3250 50  0000 C CNN
+F 1 "TX/RX" H 4250 3250 50  0000 C CNN
 F 2 "Connector_PinHeader_2.54mm:PinHeader_1x02_P2.54mm_Vertical" H 4150 3150 50  0001 C CNN
 F 3 "~" H 4150 3150 50  0001 C CNN
@@
 P 8800 4300
 F 0 "J3" H 8693 3975 50  0000 C CNN
-F 1 "Distance sensor 2" H 8693 4066 50  0000 C CNN
+F 1 "sensor 2" H 8693 4066 50  0000 C CNN
 F 2 "Connector_PinSocket_2.54mm:PinSocket_1x03_P2.54mm_Vertical" H 8800 4300 50  0001 C CNN
 F 3 "~" H 8800 4300 50  0001 C CNN
@@
 P 8800 5300
 F 0 "J5" H 8693 4975 50  0000 C CNN
-F 1 "Distance sensor 3" H 8693 5066 50  0000 C CNN
+F 1 "sensor 3" H 8693 5066 50  0000 C CNN
 F 2 "Connector_PinSocket_2.54mm:PinSocket_1x03_P2.54mm_Vertical" H 8800 5300 50  0001 C CNN
 F 3 "~" H 8800 5300 50  0001 C CNN
@@
 P 10600 3300
 F 0 "J7" H 10493 2975 50  0000 C CNN
-F 1 "Distance sensor 4" H 10493 3066 50  0000 C CNN
+F 1 "sensor 4" H 10493 3066 50  0000 C CNN
 F 2 "Connector_PinSocket_2.54mm:PinSocket_1x03_P2.54mm_Vertical" H 10600 3300 50  0001 C CNN
 F 3 "~" H 10600 3300 50  0001 C CNN
@@
 P 10600 4300
 F 0 "J8" H 10493 3975 50  0000 C CNN
-F 1 "Distance sensor 5" H 10493 4066 50  0000 C CNN
+F 1 "sensor 5" H 10493 4066 50  0000 C CNN
 F 2 "Connector_PinSocket_2.54mm:PinSocket_1x03_P2.54mm_Vertical" H 10600 4300 50  0001 C CNN
 F 3 "~" H 10600 4300 50  0001 C CNN
